Commit message: fail to load controllers

File: urdf/kr210.gazebo.xacro (robot description, xacro)
@@ -1,84 +1,39 @@
 <?xml version="1.0"?>
-<robot>
-  <!-- Link0 -->
-  <gazebo reference="base_link">
-    <material>Gazebo/Grey</material>
-    <mu1>2</mu1>
-    <mu2>2</mu2>
-  </gazebo>
-  <!-- Link1 -->
-  <gazebo reference="link_1">
-    <mu1>0.2</mu1>
-    <mu2>0.2</mu2>
-  </gazebo>
-  <!-- Link2 -->
-  <gazebo reference="link_2">
-    <mu1>0.2</mu1>
-    <mu2>0.2</mu2>
-  </gazebo>
-  <!-- Link3 -->
-  <gazebo reference="link_3">
-    <mu1>0.2</mu1>
-    <mu2>0.2</mu2>
-  </gazebo>
-  <!-- Link4 -->
-  <gazebo reference="link_4">
-    <mu1>0.2</mu1>
-    <mu2>0.2</mu2>
-  </gazebo>
-  <!-- Link5 -->
-  <gazebo reference="link_5">
-    <mu1>0.2</mu1>
-    <mu2>0.2</mu2>
-  </gazebo>
-  <!-- Link6 -->
-  <gazebo reference="link_6">
-    <mu1>0.2</mu1>
-    <mu2>0.2</mu2>
-  </gazebo>
-  <!-- Gripper -->
-  <gazebo reference="gripper_link">
-    <material>Gazebo/Grey</material>
-    <mu1>0.2</mu1>
-    <mu2>0.2</mu2>
-  </gazebo>
-  <gazebo reference="left_gripper_finger_link">
-    <material>Gazebo/Grey</material>
-    <kp>1000000.0</kp>
-    <kd>1.0</kd>
-    <mu1>30.0</mu1>
-    <mu2>30.0</mu2>
-  </gazebo>
-  <gazebo reference="right_gripper_finger_link">
-    <material>Gazebo/Grey</material>
-    <kp>1000000.0</kp>
-    <kd>1.0</kd>
-    <mu1>30.0</mu1>
-    <mu2>30.0</mu2>
-  </gazebo>
-  <!-- ros_control plugin -->
-  <gazebo>
-    <plugin name="gazebo_ros_control" filename="libgazebo_ros_control.so">
-      <robotNamespace>/kuka_robot</robotNamespace>
-      <robotSimType>gazebo_ros_control/DefaultRobotHWSim</robotSimType>
-    </plugin>
-  </gazebo>
-  <!-- grasp plugin -->
-  <gazebo>
-    <plugin name="gazebo_grasp_fix" filename="libgazebo_grasp_fix.so">
-      <arm>
-        <arm_name>kuka_robot</arm_name>
-        <palm_link>link_6</palm_link>
-        <gripper_link>right_gripper_finger_link</gripper_link>
-        <gripper_link>left_gripper_finger_link</gripper_link>
-      </arm>
-      <forces_angle_tolerance>100</forces_angle_tolerance>
-      <update_rate>4</update_rate>
-      <grip_count_threshold>4</grip_count_threshold>
-      <max_grip_count>8</max_grip_count>
-      <release_tolerance>0.003</release_tolerance>
-      <disable_collisions_on_attach>false</disable_collisions_on_attach>
-      <contact_topic>__default_topic__</contact_topic>
-    </plugin>
-  </gazebo>
+<robot xmlns:xacro="http://wiki.ros.org/xacro">
+  <ros2_control name="GazeboSystem" type="system">
+    <hardware>
+      <plugin>gazebo_ros2_control/GazeboSystem</plugin>
+    </hardware>
+    <!-- ARM JOINTS -->
+    <joint name="joint_1">
+      <command_interface name="position"/>
+      <state_interface name="position"/>
+      <state_interface name="velocity"/>
+    </joint>
+    <joint name="joint_2">
+      <command_interface name="position"/>
+      <state_interface name="position"/>
+      <state_interface name="velocity"/>
+    </joint>
+    <joint name="joint_3">
+      <command_interface name="position"/>
+      <state_interface name="position"/>
+      <state_interface name="velocity"/>
+    </joint>
+    <joint name="joint_4">
+      <command_interface name="position"/>
+      <state_interface name="position"/>
+      <state_interface name="velocity"/>
+    </joint>
+    <joint name="joint_5">
+      <command_interface name="position"/>
+      <state_interface name="position"/>
+      <state_interface name="velocity"/>
+    </joint>
+    <joint name="joint_6">
+      <command_interface name="position"/>
+      <state_interface name="position"/>
+      <state_interface name="velocity"/>
+    </joint>
+  </ros2_control>
 </robot>

File: urdf/kr210.urdf.xacro (robot description, xacro)
@@ -15,4 +15,9 @@
   <xacro:property name="gripper_type" value="two_finger" /><!--value="vacuum" or "two_finger"-->
   <xacro:property name="vacuum_gripper_radius" value="0.1" />
+    <gazebo>
+        <plugin name="gazebo_ros2_control" filename="libgazebo_ros2_control.so">
+            <parameters>$(find kuka_robot)/config/controllers.yaml</parameters>
+        </plugin>
+    </gazebo>
   <!--Import gazebo elements-->
   <xacro:include filename="$(find kuka_robot)/urdf/kr210.gazebo.xacro" />
@@ -28,14 +33,14 @@
       <origin xyz="0 0 0" rpy="${-pi/2} 0 0"/>
       <geometry>
-        <mesh filename="package://kuka_robot/meshes/kr210l150/visual/base_link.dae"/>
-      </geometry>
-      <material name="">
-        <color rgba="0.75294 0.75294 0.75294 1"/>
-      </material>
-    </visual>
-    <collision>
-      <origin xyz="0 0 0" rpy="${-pi/2} 0 0"/>
-      <geometry>
-        <mesh filename="package://kuka_robot/meshes/kr210l150/collision/base_link.stl"/>
+        <mesh filename="file://$(find kuka_robot)/meshes/kr210l150/visual/base_link.dae"/>
+      </geometry>
+      <material name="">
+        <color rgba="0.75294 0.75294 0.75294 1"/>
+      </material>
+    </visual>
+    <collision>
+      <origin xyz="0 0 0" rpy="${-pi/2} 0 0"/>
+      <geometry>
+        <mesh filename="file://$(find kuka_robot)/meshes/kr210l150/collision/base_link.stl"/>
       </geometry>
     </collision>
@@ -50,14 +55,14 @@
       <origin xyz="0 0 0" rpy="0 0 0"/>
       <geometry>
-        <mesh filename="package://kuka_robot/meshes/kr210l150/visual/link_1.dae"/>
-      </geometry>
-      <material name="">
-        <color rgba="0.75294 0.75294 0.75294 1"/>
-      </material>
-    </visual>
-    <collision>
-      <origin xyz="0 0 0" rpy="0 0 0"/>
-      <geometry>
-        <mesh filename="package://kuka_robot/meshes/kr210l150/collision/link_1.stl"/>
+        <mesh filename="file://$(find kuka_robot)/meshes/kr210l150/visual/link_1.dae"/>
+      </geometry>
+      <material name="">
+        <color rgba="0.75294 0.75294 0.75294 1"/>
+      </material>
+    </visual>
+    <collision>
+      <origin xyz="0 0 0" rpy="0 0 0"/>
+      <geometry>
+        <mesh filename="file://$(find kuka_robot)/meshes/kr210l150/collision/link_1.stl"/>
       </geometry>
     </collision>
@@ -72,14 +77,14 @@
       <origin xyz="0 0 0" rpy="${-pi/2} 0 0"/>
       <geometry>
-        <mesh filename="package://kuka_robot/meshes/kr210l150/visual/link_2.dae"/>
-      </geometry>
-      <material name="">
-        <color rgba="0.75294 0.75294 0.75294 1"/>
-      </material>
-    </visual>
-    <collision>
-      <origin xyz="0 0 0" rpy="0 0 0"/>
-      <geometry>
-        <mesh filename="package://kuka_robot/meshes/kr210l150/collision/link_2.stl"/>
+        <mesh filename="file://$(find kuka_robot)/meshes/kr210l150/visual/link_2.dae"/>
+      </geometry>
+      <material name="">
+        <color rgba="0.75294 0.75294 0.75294 1"/>
+      </material>
+    </visual>
+    <collision>
+      <origin xyz="0 0 0" rpy="0 0 0"/>
+      <geometry>
+        <mesh filename="file://$(find kuka_robot)/meshes/kr210l150/collision/link_2.stl"/>
       </geometry>
     </collision>
@@ -94,5 +99,5 @@
       <origin xyz="0 -0.184 0" rpy="${-pi/2} 0 0"/>
       <geometry>
-        <mesh filename="package://kuka_robot/meshes/kr210l150/visual/link_3.dae"/>
+        <mesh filename="file://$(find kuka_robot)/meshes/kr210l150/visual/link_3.dae"/>
       </geometry>
       <material name="">
@@ -103,5 +108,5 @@
       <origin xyz="0 -0.184 0" rpy="0 0 0"/>
       <geometry>
-        <mesh filename="package://kuka_robot/meshes/kr210l150/collision/link_3.stl"/>
+        <mesh filename="file://$(find kuka_robot)/meshes/kr210l150/collision/link_3.stl"/>
       </geometry>
     </collision>
@@ -116,14 +121,14 @@
       <origin xyz="0 0 0" rpy="${-pi/2} 0 0"/>
       <geometry>
-        <mesh filename="package://kuka_robot/meshes/kr210l150/visual/link_4.dae"/>
-      </geometry>
-      <material name="">
-        <color rgba="0.75294 0.75294 0.75294 1"/>
-      </material>
-    </visual>
-    <collision>
-      <origin xyz="0 0 0" rpy="0 0 0"/>
-      <geometry>
-        <mesh filename="package://kuka_robot/meshes/kr210l150/collision/link_4.stl"/>
+        <mesh filename="file://$(find kuka_robot)/meshes/kr210l150/visual/link_4.dae"/>
+      </geometry>
+      <material name="">
+        <color rgba="0.75294 0.75294 0.75294 1"/>
+      </material>
+    </visual>
+    <collision>
+      <origin xyz="0 0 0" rpy="0 0 0"/>
+      <geometry>
+        <mesh filename="file://$(find kuka_robot)/meshes/kr210l150/collision/link_4.stl"/>
       </geometry>
     </collision>
@@ -138,14 +143,14 @@
       <origin xyz="0 0 0" rpy="${-pi/2} 0 0"/>
       <geometry>
-        <mesh filename="package://kuka_robot/meshes/kr210l150/visual/link_5.dae"/>
-      </geometry>
-      <material name="">
-        <color rgba="0.75294 0.75294 0.75294 1"/>
-      </material>
-    </visual>
-    <collision>
-      <origin xyz="0 0 0" rpy="0 0 0"/>
-      <geometry>
-        <mesh filename="package://kuka_robot/meshes/kr210l150/collision/link_5.stl"/>
+        <mesh filename="file://$(find kuka_robot)/meshes/kr210l150/visual/link_5.dae"/>
+      </geometry>
+      <material name="">
+        <color rgba="0.75294 0.75294 0.75294 1"/>
+      </material>
+    </visual>
+    <collision>
+      <origin xyz="0 0 0" rpy="0 0 0"/>
+      <geometry>
+        <mesh filename="file://$(find kuka_robot)/meshes/kr210l150/collision/link_5.stl"/>
       </geometry>
     </collision>
@@ -160,14 +165,14 @@
       <origin xyz="0 0 0" rpy="0 0 0"/>
       <geometry>
-        <mesh filename="package://kuka_robot/meshes/kr210l150/visual/link_6.dae"/>
-      </geometry>
-      <material name="">
-        <color rgba="0.75294 0.75294 0.75294 1"/>
-      </material>
-    </visual>
-    <collision>
-      <origin xyz="0 0 0" rpy="0 0 0"/>
-      <geometry>
-        <mesh filename="package://kuka_robot/meshes/kr210l150/collision/link_6.stl"/>
+        <mesh filename="file://$(find kuka_robot)/meshes/kr210l150/visual/link_6.dae"/>
+      </geometry>
+      <material name="">
+        <color rgba="0.75294 0.75294 0.75294 1"/>
+      </material>
+    </visual>
+    <collision>
+      <origin xyz="0 0 0" rpy="0 0 0"/>
+      <geometry>
+        <mesh filename="file://$(find kuka_robot)/meshes/kr210l150/collision/link_6.stl"/>
       </geometry>
     </collision>
@@ -212,11 +217,11 @@
       <origin xyz="0 0 0" rpy="0 0 0"/>
       <geometry>
-        <mesh filename="package://kuka_robot/meshes/gripper/gripper_base.dae"/>
-      </geometry>
-    </visual>
-    <collision>
-      <origin xyz="0 0 0" rpy="0 0 0"/>
-      <geometry>
-        <mesh filename="package://kuka_robot/meshes/gripper/gripper_base.dae"/>
+        <mesh filename="file://$(find kuka_robot)/meshes/gripper/gripper_base.dae"/>
+      </geometry>
+    </visual>
+    <collision>
+      <origin xyz="0 0 0" rpy="0 0 0"/>
+      <geometry>
+        <mesh filename="file://$(find kuka_robot)/meshes/gripper/gripper_base.dae"/>
       </geometry>
     </collision>
@@ -231,11 +236,11 @@
       <origin xyz="0 0 0" rpy="0 0 0"/>
       <geometry>
-        <mesh filename="package://kuka_robot/meshes/gripper/finger_right.dae"/>
-      </geometry>
-    </visual>
-    <collision>
-      <origin xyz="0 0 0" rpy="0 0 0"/>
-      <geometry>
-        <mesh filename="package://kuka_robot/meshes/gripper/finger_right_collision.dae"/>
+        <mesh filename="file://$(find kuka_robot)/meshes/gripper/finger_right.dae"/>
+      </geometry>
+    </visual>
+    <collision>
+      <origin xyz="0 0 0" rpy="0 0 0"/>
+      <geometry>
+        <mesh filename="file://$(find kuka_robot)/meshes/gripper/finger_right_collision.dae"/>
       </geometry>
     </collision>
@@ -250,11 +255,11 @@
       <origin xyz="0 0 0" rpy="0 0 0"/>
       <geometry>
-        <mesh filename="package://kuka_robot/meshes/gripper/finger_left.dae"/>
-      </geometry>
-    </visual>
-    <collision>
-      <origin xyz="0 0 0" rpy="0 0 0"/>
-      <geometry>
-        <mesh filename="package://kuka_robot/meshes/gripper/finger_left_collision.dae"/>
+        <mesh filename="file://$(find kuka_robot)/meshes/gripper/finger_left.dae"/>
+      </geometry>
+    </visual>
+    <collision>
+      <origin xyz="0 0 0" rpy="0 0 0"/>
+      <geometry>
+        <mesh filename="file://$(find kuka_robot)/meshes/gripper/finger_left_collision.dae"/>
       </geometry>
     </collision>
@@ -282,24 +287,4 @@
     <axis xyz="0 1 0" />
   </joint>
-  <transmission name="tran7">
-    <type>transmission_interface/SimpleTransmission</type>
-    <joint name="left_gripper_finger_joint">
-      <hardwareInterface>hardware_interface/EffortJointInterface</hardwareInterface>
-    </joint>
-    <actuator name="motor7">
-      <hardwareInterface>hardware_interface/EffortJointInterface</hardwareInterface>
-      <mechanicalReduction>1</mechanicalReduction>
-    </actuator>
-  </transmission>
-  <transmission name="tran8">
-    <type>transmission_interface/SimpleTransmission</type>
-    <joint name="right_gripper_finger_joint">
-      <hardwareInterface>hardware_interface/EffortJointInterface</hardwareInterface>
-    </joint>
-    <actuator name="motor8">
-      <hardwareInterface>hardware_interface/EffortJointInterface</hardwareInterface>
-      <mechanicalReduction>1</mechanicalReduction>
-    </actuator>
-  </transmission>
   </xacro:if>
   <!-- joints -->
@@ -351,64 +336,3 @@
     <limit lower="${-350*deg}" upper="${350*deg}" effort="300" velocity="${219*deg}"/>
   </joint>
-  <!--Transmission and actuators-->
-  <transmission name="tran1">
-    <type>transmission_interface/SimpleTransmission</type>
-    <joint name="joint_1">
-      <hardwareInterface>hardware_interface/PositionJointInterface</hardwareInterface>
-    </joint>
-    <actuator name="motor1">
-      <hardwareInterface>hardware_interface/PositionJointInterface</hardwareInterface>
-      <mechanicalReduction>1</mechanicalReduction>
-    </actuator>
-  </transmission>
-  <transmission name="tran2">
-    <type>transmission_interface/SimpleTransmission</type>
-    <joint name="joint_2">
-      <hardwareInterface>hardware_interface/PositionJointInterface</hardwareInterface>
-    </joint>
-    <actuator name="motor2">
-      <hardwareInterface>hardware_interface/PositionJointInterface</hardwareInterface>
-      <mechanicalReduction>1</mechanicalReduction>
-    </actuator>
-  </transmission>
-  <transmission name="tran3">
-    <type>transmission_interface/SimpleTransmission</type>
-    <joint name="joint_3">
-      <hardwareInterface>hardware_interface/PositionJointInterface</hardwareInterface>
-    </joint>
-    <actuator name="motor3">
-      <hardwareInterface>hardware_interface/PositionJointInterface</hardwareInterface>
-      <mechanicalReduction>1</mechanicalReduction>
-    </actuator>
-  </transmission>
-  <transmission name="tran4">
-    <type>transmission_interface/SimpleTransmission</type>
-    <joint name="joint_4">
-      <hardwareInterface>hardware_interface/PositionJointInterface</hardwareInterface>
-    </joint>
-    <actuator name="motor4">
-      <hardwareInterface>hardware_interface/PositionJointInterface</hardwareInterface>
-      <mechanicalReduction>1</mechanicalReduction>
-    </actuator>
-  </transmission>
-  <transmission name="tran5">
-    <type>transmission_interface/SimpleTransmission</type>
-    <joint name="joint_5">
-      <hardwareInterface>hardware_interface/PositionJointInterface</hardwareInterface>
-    </joint>
-    <actuator name="motor5">
-      <hardwareInterface>hardware_interface/PositionJointInterface</hardwareInterface>
-      <mechanicalReduction>1</mechanicalReduction>
-    </actuator>
-  </transmission>
-  <transmission name="tran6">
-    <type>transmission_interface/SimpleTransmission</type>
-    <joint name="joint_6">
-      <hardwareInterface>hardware_interface/PositionJointInterface</hardwareInterface>
-    </joint>
-    <actuator name="motor6">
-      <hardwareInterface>hardware_interface/PositionJointInterface</hardwareInterface>
-      <mechanicalReduction>1</mechanicalReduction>
-    </actuator>
-  </transmission>
 </robot>

Commit message: managed to load controllers the system needed reboot

File: urdf/kr210.gazebo.xacro (robot description, xacro)
@@ -36,4 +36,20 @@
       <state_interface name="velocity"/>
     </joint>
+    <!-- GRIPPER -->
+    <joint name="right_gripper_finger_joint">
+      <command_interface name="position"/>
+      <state_interface name="position"/>
+      <state_interface name="velocity"/>
+    </joint>
+    <joint name="left_gripper_finger_joint">
+      <command_interface name="position"/>
+      <state_interface name="position"/>
+      <state_interface name="velocity"/>
+    </joint>
   </ros2_control>
+    <gazebo>
+        <plugin name="gazebo_ros2_control" filename="libgazebo_ros2_control.so">
+            <parameters>$(find kuka_robot)/config/controllers.yaml</parameters>
+        </plugin>
+    </gazebo>
 </robot>

File: urdf/kr210.urdf.xacro (robot description, xacro)
@@ -15,9 +15,4 @@
   <xacro:property name="gripper_type" value="two_finger" /><!--value="vacuum" or "two_finger"-->
   <xacro:property name="vacuum_gripper_radius" value="0.1" />
-    <gazebo>
-        <plugin name="gazebo_ros2_control" filename="libgazebo_ros2_control.so">
-            <parameters>$(find kuka_robot)/config/controllers.yaml</parameters>
-        </plugin>
-    </gazebo>
   <!--Import gazebo elements-->
   <xacro:include filename="$(find kuka_robot)/urdf/kr210.gazebo.xacro" />
